Commit message: L1BR seguiu trajetoria

File: src/robot_description/urdf/robot_parts/carcaca.xacro (robot description, xacro)
@@ -6,13 +6,15 @@
             <mu1 value="0.3" />
             <mu2 value="0.3" />
-            <kp value="10000000.0" />
-            <kd value="1000" />
+            <kp value="1000000.0" />
+            <kd value="100" />
             <fdir1 value="0 0 0" />
         </gazebo>
         <link name="${base_link}">
             <inertial>
-                <mass value="15" />
+                <mass value="2.4" />
                 <origin rpy="0  0  3.14" xyz="0  0  0.0118" />
-                <inertia ixx="1" ixy="0" ixz="0" iyy="1" iyz="0" izz="1" />
+                <inertia ixx="0.019995" ixy="0.0" ixz="0.0"
+                iyy="0.019995" iyz="0.0"
+                izz="0.03675" />
             </inertial>
             <collision name="${base_link}_collision">

File: src/robot_description/urdf/robot_parts/traction_wheel.xacro (robot description, xacro)
@@ -11,8 +11,10 @@
         <gazebo reference="${prefix}">
             <selfCollide>false</selfCollide>
-            <mu1 value="100" />
-            <mu2 value="50" />
-            <kp value="10000000.0" />
-            <kd value="1000" />
+            <mu1>1.0</mu1>
+            <mu2>1.0</mu2>
+            <kp>1000000.0</kp>
+            <kd>100.0</kd>
+            <minDepth>0.001</minDepth>
+            <maxVel>1.0</maxVel>
             <fdir1 value="0 0 0" />
         </gazebo>
@@ -21,5 +23,7 @@
                 <mass value="1" />
                 <origin rpy="0 0 0" xyz="0 0 0" />
-                <inertia ixx="1" ixy="0" ixz="0" iyy="1" iyz="0" izz="1" />
+                <inertia ixx="0.001" ixy="0.0" ixz="0.0"
+                iyy="0.001" iyz="0.0"
+                izz="0.001" />
             </inertial>
             <collision name="${prefix}_collision">
